File: pcb/HDMI-Display_v10dev.brd (EAGLE design)
At the start: 52 x 52 mm, 95 parts, among them IC1 TFP401A-PAD, IC2 24LC02B, IC3 IS31BL3506A-TTLS2, IC4 ATMEGA32U4-MU, IC5 LDO-TS1117-3V3, Q1 16MHz, SW1 SW-TACTILE-TL3315, X1 PASSER-07, X2 PASSER-07, X3 PASSER-07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

Commit message: updated schematics
Parts:
- R7B: value 100k -> NM
Changed lines of the file:
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@@
 <setting verticaltext="up"/>
 </settings>
-<grid distance="0.05" unitdist="inch" unit="inch" style="lines" multiple="1" display="yes" altdistance="0.0125" altunitdist="inch" altunit="inch"/>
+<grid distance="0.05" unitdist="inch" unit="inch" style="lines" multiple="1" display="yes" altdistance="0.025" altunitdist="inch" altunit="inch"/>
 <layers>
 <layer number="1" name="Top" color="4" fill="1" visible="yes" active="yes"/>
@@
 <attribute name="NAME" x="22.86" y="13.335" size="0.8128" layer="21" font="vector" ratio="10" align="center"/>
 </element>
-<element name="R7B" library="we-rcl" package="R0402" value="100k" x="4.1275" y="16.03375" smashed="yes" rot="R180">
+<element name="R7B" library="we-rcl" package="R0402" value="NM" x="4.1275" y="16.03375" smashed="yes" rot="R180">
 <attribute name="NAME" x="5.23875" y="16.03375" size="0.8128" layer="25" font="vector" ratio="10" rot="R270" align="center"/>
 <attribute name="VALUE" x="2.8575" y="16.03375" size="0.8128" layer="27" font="vector" ratio="10" rot="R90" align="center"/>
