File: pcb/HDMI-Display_v10.sch (EAGLE design)
At the start: 95 parts, among them IC1 TFP401A-PAD, IC2 24LC02B, IC3 IS31BL3506A-TTLS2, IC4 ATMEGA32U4-MU, IC5 LDO-TS1117-3V3, Q1 16MHz, SW1 SW-TACTILE-TL3315, X1 PASSER-07, X2 PASSER-07, X3 PASSER-07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

Commit message: updated layout and schematics
Parts:
- removed 40MA: JUMPER2, we-rcl:JUMPER2
- removed LCD: ER-TFT050-3, we-opto:ER-TFT050-3
- removed LCD2: FPC40, we-con:FPC40
- removed X+, X-, Y+, Y-: PAD-0.80X1.60_NC, we-rcl:PAD-0.80X1.60_NC
- added J20_1, J20_2, TP_INT, TP_SCL, TP_SDA: JUMPER2-0402, we-rcl:JUMPER2-0402
- added LCD_BOT: FPC40, we-con:FPC40
- added LCD_TOP: ER-TFT050-3, we-opto:ER-TFT050-3
- added R7: NM, we-rcl:RESISTOR-R0402
- added RS3: 15, we-rcl:RESISTOR-R0402
- added TP: FPC06, we-con:FPC06
- added TP_BOT: FPC04, we-con:FPC04
- 3V3, 5V, GND: value PAD-1.27X2.54_NC -> PAD-1.27X1.27_NC; device we-rcl:PAD-1.27X2.54_NC -> we-rcl:PAD-1.27X1.27_NC
- C17: value 10nF -> 100n
- C18: value 100nF -> 4u7
- C20, C21: value 100nF -> 100n
- C6: value 100n -> 4u7
- HPWR, SCL, SDA: value JUMPER2 -> JUMPER2-0603; device we-rcl:JUMPER2 -> we-rcl:JUMPER2-0603
- L1: value 10u@500mA -> 10u @ 500mA
- OCK-INV: value JUMPER2 -> JUMPER2-0603-NC; device we-rcl:JUMPER2 -> we-rcl:JUMPER2-0603-NC
- PWR: value JUMPER3 -> JUMPER3-0603; device we-rcl:JUMPER3 -> we-rcl:JUMPER3-0603
- T1, T2, T3, T4, T5: value (none) -> BSS138
- VCCIO: value JUMPER3-NOCREAM -> JUMPER3-0603-NC; device we-rcl:JUMPER3-NOCREAM -> we-rcl:JUMPER3-0603-NC
Connections:
- new net LV_WAKE: TP.4
- new net N$1: J20_2.2, RS3.2
- net +3V3: now also LCD_TOP.VCC, R7.2, TP.3; no longer LCD.VCC
- net B0: now also LCD_TOP.B0; no longer LCD.B0
- net B1: now also LCD_TOP.B1; no longer LCD.B1
- net B2: now also LCD_TOP.B2; no longer LCD.B2
- net B3: now also LCD_TOP.B3; no longer LCD.B3
- net B4: now also LCD_TOP.B4; no longer LCD.B4
- net B5: now also LCD_TOP.B5; no longer LCD.B5
- net B6: now also LCD_TOP.B6; no longer LCD.B6
- net B7: now also LCD_TOP.B7; no longer LCD.B7
- net CLK: now also LCD_TOP.CLK; no longer LCD.CLK
- net DE: now also LCD_TOP.DE; no longer LCD.DE
- net G0: now also LCD_TOP.G0; no longer LCD.G0
- net G1: now also LCD_TOP.G1; no longer LCD.G1
- net G2: now also LCD_TOP.G2; no longer LCD.G2
- net G3: now also LCD_TOP.G3; no longer LCD.G3
- net G4: now also LCD_TOP.G4; no longer LCD.G4
- net G5: now also LCD_TOP.G5; no longer LCD.G5
- net G6: now also LCD_TOP.G6; no longer LCD.G6
- net G7: now also LCD_TOP.G7; no longer LCD.G7
- net GND: now also LCD_BOT.12, LCD_BOT.38, LCD_BOT.5, LCD_TOP.GND, RS3.1, TP.6; no longer LCD.GND, LCD2.12, LCD2.38, LCD2.5
- net HSYNC: now also LCD_TOP.HSYNC; no longer LCD.HSYNC
- net LED+: now also LCD_TOP.A; no longer LCD.A
- net LED-: now also J20_1.1, LCD_TOP.C; no longer 40MA.1, LCD.C
- net LV_GPIO: now also TP.5, TP_INT.2
- net LV_SCL: now also TP.1, TP_SCL.2
- net LV_SDA: now also TP.2, TP_SDA.2
- net N$4: now also J20_1.2, J20_2.1; no longer 40MA.2
- net PDO: now also LCD_TOP.DISP; no longer LCD.DISP
- net R0: now also LCD_TOP.R0; no longer LCD.R0
- net R1: now also LCD_TOP.R1; no longer LCD.R1
- net R2: now also LCD_TOP.R2; no longer LCD.R2
- net R3: now also LCD_TOP.R3; no longer LCD.R3
- net R4: now also LCD_TOP.R4; no longer LCD.R4
- net R5: now also LCD_TOP.R5; no longer LCD.R5
- net R6: now also LCD_TOP.R6; no longer LCD.R6
- net R7: now also LCD_TOP.R7; no longer LCD.R7
- net VSYNC: now also LCD_TOP.VSYNC; no longer LCD.VSYNC
- net X+: now also LCD_TOP.X+, TP_BOT.4, TP_SDA.1; no longer LCD.X+, X+.P
- net X-: now also LCD_TOP.X-, R7.1, TP_BOT.2; no longer LCD.X-, X-.P
- net Y+: now also LCD_TOP.Y+, TP_BOT.1, TP_INT.1; no longer LCD.Y+, Y+.P
- net Y-: now also LCD_TOP.Y-, TP_BOT.3, TP_SCL.1; no longer LCD.Y-, Y-.P
Other:
- note added: "6-pin I2C touch controller"
- note added: "A0"
- note added: "A1"
- note added: "A2"
- note added: "A3"
- note added: "A4"
- note added: "A5"
- note added: "D0"
- note added: "D1"
- note added: "D10"
- note added: "D11"
- note added: "D12"
- note added: "D13"
- note added: "D2"
- note added: "D3"
- note added: "D4"
- note added: "D5"
- note added: "D6"
- note added: "D7"
- note added: "D8"
- note added: "D9"
- note added: "GND"
- note added: "I2C / resistive"
- note added: "INT"
- note added: "INT /"
- note added: "MISO"
- note added: "MOSI"
- note added: "RES /"
- note added: "RxLED"
- note added: "SCK"
- note added: "SCL"
- note added: "SCL /"
- note added: "SDA"
- note added: "SDA /"
- note added: "TFT070-4 - 7" 800x480 BL:40mA TFT050-3 - 5" 800x480 BL:40mA TFT043-3 - 4.3" 480x272 BL:20mA"
- note added: "TxLED"
- note added: "VCC"
- note added: "WAK"
- note added: "ambient light sensor"
- note added: "close jumpers for I2C touch controller"
- note removed: "Ambient light sensor"
- note removed: "Developer Edition"
- moved on the sheet: C10, C11, C12, C13, C14, C15, C16, C17, C18, C6, C7, C8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
