File: pcb/HDMI-Display_v10.sch (EAGLE design)
At the start: 99 parts, among them IC1 TFP401A-PAD, IC2 24LC02B, IC3 IS31BL3506A-TTLS2, IC4 ATMEGA32U4-MU, IC5 LDO-TS1117-3V3, J20_1 JUMPER2-0402, J20_2 JUMPER2-0402, Q1 16MHz, SW1 SW-TACTILE-TL3315, T1 BSS138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

Commit message: updated schematics
Parts:
- LED1: value LED-0603 -> green
- LED2: value LED-0603 -> red
Changed lines of the file:
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@@
 <part name="GND14" library="supply1" deviceset="GND" device=""/>
 <part name="SW1" library="we-switch" deviceset="SW-TACTILE" device="-TL3315"/>
-<part name="LED1" library="we-opto" deviceset="LED" device="-0603"/>
-<part name="LED2" library="we-opto" deviceset="LED" device="-0603"/>
+<part name="LED1" library="we-opto" deviceset="LED" device="-0603" value="green"/>
+<part name="LED2" library="we-opto" deviceset="LED" device="-0603" value="red"/>
 <part name="GND3" library="supply1" deviceset="GND" device=""/>
 <part name="GND4" library="supply1" deviceset="GND" device=""/>
