File: pcb/HDMI-Display_v10.brd (EAGLE design)
At the start: 52 x 52 mm, 99 parts, among them IC1 TFP401A-PAD, IC2 24LC02B, IC3 IS31BL3506A-TTLS2, IC4 ATMEGA32U4-MU, IC5 LDO-TS1117-3V3, J20_1 JUMPER2-0402, J20_2 JUMPER2-0402, Q1 16MHz, SW1 SW-TACTILE-TL3315, T1 BSS138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

Commit message: updated schematics
Parts:
- LED1: value LED-0603 -> green
- LED2: value LED-0603 -> red
Changed lines of the file:
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@@
 <attribute name="NAME" x="22.86" y="4.1275" size="0.8128" layer="21" font="vector" ratio="10" rot="R90" align="center"/>
 </element>
-<element name="LED1" library="we-opto" package="LED_0603" value="LED-0603" x="39.37" y="9.04875" smashed="yes" rot="R180">
+<element name="LED1" library="we-opto" package="LED_0603" value="green" x="39.37" y="9.04875" smashed="yes" rot="R180">
 <attribute name="NAME" x="38.4175" y="8.89" size="0.8128" layer="25" font="vector" ratio="10" rot="R270" align="center"/>
 </element>
-<element name="LED2" library="we-opto" package="LED_0603" value="LED-0603" x="40.79875" y="9.04875" smashed="yes" rot="R180">
+<element name="LED2" library="we-opto" package="LED_0603" value="red" x="40.79875" y="9.04875" smashed="yes" rot="R180">
 <attribute name="NAME" x="41.75125" y="8.89" size="0.8128" layer="25" font="vector" ratio="10" rot="R270" align="center"/>
 </element>
