File: hardware/HDMI-Display_v13.brd (EAGLE design)
At the start: 52 x 52 mm, 107 parts, among them IC1 TFP401A-PAD, IC2 24LC02B, IC3 IS31BL3506A-TTLS2, IC4 ATMEGA32U4-MU, IC5 VREG-TS1117CW-3V3, J20_1 JUMPER2-0402, J20_2 JUMPER2-0402, J30_1 JUMPER2-0402, J30_2 JUMPER2-0402, Q1 16MHz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

Commit message: updated layout and schematics
Parts:
- USB: value USB-MICROB -> USB-MICROB-2; device we-con:USB-MICROB-10103594 -> we-con:USB-MICROB-10118194
- moved USB 0.63 mm to (50.1, 23.0)
Connections:
- net SHLD1: now also USB.SHLD3, USB.SHLD4, USB.SHLD5, USB.SHLD6, USB.SHLD7, USB.SHLD8
Routing:
- net SHLD1: track 10.0 -> 17.3 mm
- net VBUS: track 10.8 -> 11.8 mm
- net USBD_P: track 7.44 -> 8.46 mm
- net USBD_N: track 7.20 -> 8.22 mm
Other:
- board size 52 x 52 mm -> 53 x 52 mm
Changed lines of the file:
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@@
 <text x="44.92625" y="28.73375" size="0.8128" layer="21" font="vector" ratio="12" rot="R90" align="center">EDID
 Prog.</text>
+<wire x1="53" y1="51" x2="53" y2="1" width="2" layer="46"/>
 </plain>
 <attributes>
@@
 <attribute name="VALUE" x="47.81" y="37.845" size="0.8128" layer="27" font="vector" ratio="10" align="center"/>
 </element>
-<element name="USB" library="we-con" package="USB-MICROB-10103594" value="USB-MICROB" x="49.5" y="23" smashed="yes">
-<attribute name="DIGIKEY" value="609-4050-6-ND" x="49.5" y="23" size="1.778" layer="27" display="off"/>
-<attribute name="NAME" x="48.02125" y="22.93625" size="1.016" layer="21" font="vector" ratio="12" rot="R270" align="center"/>
+<element name="USB" library="we-con" package="USB-MICROB-10118194" value="USB-MICROB-2" x="50.135" y="23" smashed="yes">
+<attribute name="DIGIKEY" value="609-4618-6-ND " x="50.135" y="23" size="1.778" layer="27" display="off"/>
+<attribute name="NAME" x="48.65625" y="22.93625" size="1.016" layer="21" font="vector" ratio="12" rot="R270" align="center"/>
 </element>
 <element name="IC3" library="we-power" package="SOT23-6" value="IS31BL3506A-TTLS2" x="7.14375" y="14.44625" smashed="yes" rot="R180">
@@
 <wire x1="42.3125" y1="24.923025" x2="42.545" y2="25.155525" width="0.1524" layer="1"/>
 <wire x1="42.3125" y1="24.926875" x2="42.3125" y2="24.923025" width="0.1524" layer="1"/>
-<wire x1="46.615" y1="23" x2="45.7324" y2="23" width="0.1524" layer="1"/>
+<wire x1="47.635" y1="23" x2="45.7324" y2="23" width="0.1524" layer="1"/>
 <wire x1="45.7324" y1="23" x2="44.9199" y2="23.8125" width="0.1524" layer="1" curve="-90"/>
 <wire x1="42.06875" y1="24.679275" x2="41.066975" y2="24.679275" width="0.1524" layer="1"/>
@@
 <wire x1="42.31" y1="24.126875" x2="42.53865" y2="23.898225" width="0.1524" layer="1"/>
 <wire x1="42.3125" y1="24.126875" x2="42.31" y2="24.126875" width="0.1524" layer="1"/>
-<wire x1="46.615" y1="22.35" x2="45.2775" y2="22.35" width="0.1524" layer="1"/>
+<wire x1="47.635" y1="22.35" x2="45.2775" y2="22.35" width="0.1524" layer="1"/>
 <wire x1="45.2775" y1="22.35" x2="44.45" y2="23.1775" width="0.1524" layer="1" curve="-90"/>
 <wire x1="42.06875" y1="24.374475" x2="41.066975" y2="24.374475" width="0.1524" layer="1"/>
@@
 <wire x1="45.72" y1="13.1825" x2="45.71375" y2="13.1825" width="0.4064" layer="1"/>
 <wire x1="45.71375" y1="13.1825" x2="44.45" y2="14.44625" width="0.8128" layer="1"/>
-<wire x1="46.615" y1="21.7" x2="45.195" y2="21.7" width="0.4064" layer="1"/>
+<wire x1="47.635" y1="21.7" x2="45.195" y2="21.7" width="0.4064" layer="1"/>
 <wire x1="45.195" y1="21.7" x2="45.085" y2="21.59" width="0.4064" layer="1"/>
 <wire x1="45.085" y1="21.59" x2="44.45" y2="20.955" width="0.6096" layer="1"/>
@@
 <contactref element="USB" pad="SHLD2"/>
 <contactref element="R17" pad="2"/>
-<wire x1="48.26" y1="18.0975" x2="49.2125" y2="19.05" width="0.4064" layer="1"/>
-<wire x1="49.2125" y1="19.05" x2="49.2125" y2="22.06625" width="0.4064" layer="1"/>
-<wire x1="49.2125" y1="22.06625" x2="49.2125" y2="23.97125" width="0.4064" layer="1"/>
-<wire x1="49.2125" y1="23.97125" x2="49.2125" y2="26.19375" width="0.4064" layer="1"/>
-<wire x1="47.8075" y1="18.0975" x2="48.26" y2="18.0975" width="0.4064" layer="1"/>
-<wire x1="49.75" y1="23.9625" x2="49.22125" y2="23.9625" width="0.2032" layer="1"/>
-<wire x1="49.22125" y1="23.9625" x2="49.2125" y2="23.97125" width="0.2032" layer="1"/>
-<wire x1="49.75" y1="22.0375" x2="49.24125" y2="22.0375" width="0.2032" layer="1"/>
-<wire x1="49.24125" y1="22.0375" x2="49.2125" y2="22.06625" width="0.2032" layer="1"/>
+<contactref element="USB" pad="SHLD3"/>
+<contactref element="USB" pad="SHLD4"/>
+<contactref element="USB" pad="SHLD5"/>
+<contactref element="USB" pad="SHLD6"/>
+<contactref element="USB" pad="SHLD7"/>
+<contactref element="USB" pad="SHLD8"/>
+<wire x1="47.8075" y1="18.0975" x2="49.5935" y2="18.0975" width="0.4064" layer="1"/>
+<wire x1="49.657" y1="19.493" x2="50.285" y2="19.5" width="0.4064" layer="1"/>
+<wire x1="50.285" y1="19.5" x2="50.285" y2="20.15" width="0.4064" layer="1"/>
+<wire x1="50.285" y1="20.15" x2="50.285" y2="22" width="0.4064" layer="1"/>
+<wire x1="50.285" y1="22" x2="50.285" y2="24" width="0.4064" layer="1"/>
+<wire x1="50.285" y1="24" x2="50.285" y2="25.85" width="0.4064" layer="1"/>
+<wire x1="50.285" y1="26.5" x2="50.285" y2="25.85" width="0.4064" layer="1"/>
+<wire x1="49.5935" y1="18.0975" x2="50.292" y2="18.796" width="0.4064" layer="1"/>
+<wire x1="50.292" y1="18.796" x2="50.292" y2="19.493" width="0.4064" layer="1"/>
+<wire x1="50.292" y1="19.493" x2="50.285" y2="19.5" width="0.4064" layer="1"/>
+<wire x1="47.585" y1="20.45" x2="48.535" y2="19.5" width="0.4064" layer="1"/>
+<wire x1="48.535" y1="19.5" x2="50.285" y2="19.5" width="0.4064" layer="1"/>
+<wire x1="47.585" y1="25.55" x2="48.535" y2="26.5" width="0.4064" layer="1"/>
+<wire x1="48.535" y1="26.5" x2="50.285" y2="26.5" width="0.4064" layer="1"/>
 </signal>
 <signal name="LV_GPIO">
