File: hardware/HDMI-Display_v13.sch (EAGLE design)
At the start: 107 parts, among them IC1 TFP401A-PAD, IC2 24LC02B, IC3 IS31BL3506A-TTLS2, IC4 ATMEGA32U4-MU, IC5 VREG-TS1117CW-3V3, J20_1 JUMPER2-0402, J20_2 JUMPER2-0402, J30_1 JUMPER2-0402, J30_2 JUMPER2-0402, Q1 16MHz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

Commit message: updated layout and schematics
Parts:
- USB: value USB-MICROB -> USB-MICROB-2; device we-con:USB-MICROB -> we-con:USB-MICROB-2
Changed lines of the file:
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@@
 <part name="IC2" library="we-chip" deviceset="24LC*" device="-I/OT" value="24LC02B"/>
 <part name="HDMI" library="we-con" deviceset="HDMI" device="-A"/>
-<part name="USB" library="we-con" deviceset="USB" device="-MICROB"/>
+<part name="USB" library="we-con" deviceset="USB" device="-MICROB-2" value="USB-MICROB-2"/>
 <part name="IC3" library="we-power" deviceset="IS31BL3506A" device="-TTLS2"/>
 <part name="L1" library="we-power" deviceset="INDUCTOR" device="-1212" value="10u/0.5A"/>
